Commit message: update x2/x3 urdf xml ,add motion visualize in mujoco,csv2amptxt

File: robot_description/x2/x2.urdf (robot description, URDF)
Before this commit: robot x2, 23 links, 22 joints
Links:
- removed link L_ankle_pitch_link
- removed link L_elbow_pitch_link
- removed link L_hip_pitch_link
- removed link L_hip_roll_link
- removed link L_hip_yaw_link
- removed link L_knee_pitch_link
- removed link L_shoulder_pitch_link
- removed link L_shoulder_roll_link
- removed link L_shoulder_yaw_link
- removed link R_ankle_pitch_link
- removed link R_elbow_pitch_link
- removed link R_hip_pitch_link
- removed link R_hip_roll_link
- removed link R_hip_yaw_link
- removed link R_knee_pitch_link
- removed link R_shoulder_pitch_link
- removed link R_shoulder_roll_link
- removed link R_shoulder_yaw_link
- removed link pelvis_link
- added link left_ankle_pitch_link, mass 0.8; collision box size=0.23 0.07 0.02; collision sphere radius=0.005
- added link left_elbow_link, mass 0.576; collision mesh filename=meshes/left_elbow_link.STL; visual mesh filename=meshes/left_elbow_link.STL
- added link left_hip_pitch_link, mass 1.8; collision mesh filename=meshes/left_hip_pitch_link.STL; visual mesh filename=meshes/left_hip_pitch_link.STL
- added link left_hip_roll_link, mass 2.667; collision mesh filename=meshes/left_hip_roll_link.STL; visual mesh filename=meshes/left_hip_roll_link.STL
- added link left_hip_yaw_link, mass 0.841; visual mesh filename=meshes/left_hip_yaw_link.STL
- added link left_knee_link, mass 1.125; collision mesh filename=meshes/left_knee_link.STL; visual mesh filename=meshes/left_knee_link.STL
- added link left_shoulder_pitch_link, mass 0.276; collision mesh filename=meshes/left_shoulder_pitch_link.STL; visual mesh filename=meshes/left_shoulder_pitch_link.STL
- added link left_shoulder_roll_link, mass 1.126; collision mesh filename=meshes/left_shoulder_roll_link.STL; visual mesh filename=meshes/left_shoulder_roll_link.STL
- added link left_shoulder_yaw_link, mass 0.896; collision mesh filename=meshes/left_shoulder_yaw_link.STL; visual mesh filename=meshes/left_shoulder_yaw_link.STL
- added link left_wrist_roll_link, mass 0.692; collision mesh filename=meshes/left_wrist_roll_link.STL; visual mesh filename=meshes/left_wrist_roll_link.STL
- added link pelvis, mass 0.9; collision mesh filename=meshes/pelvis.STL; visual mesh filename=meshes/pelvis.STL
- added link right_ankle_pitch_link, mass 0.8; collision box size=0.23 0.07 0.02; collision sphere radius=0.005
- added link right_elbow_link, mass 0.576; collision mesh filename=meshes/right_elbow_link.STL; visual mesh filename=meshes/right_elbow_link.STL
- added link right_hip_pitch_link, mass 1.8; collision mesh filename=meshes/right_hip_pitch_link.STL; visual mesh filename=meshes/right_hip_pitch_link.STL
- added link right_hip_roll_link, mass 2.667; collision mesh filename=meshes/right_hip_roll_link.STL; visual mesh filename=meshes/right_hip_roll_link.STL
- added link right_hip_yaw_link, mass 0.947; collision mesh filename=meshes/right_hip_yaw_link.STL; visual mesh filename=meshes/right_hip_yaw_link.STL
- added link right_knee_link, mass 1.125; collision mesh filename=meshes/right_knee_link.STL; visual mesh filename=meshes/right_knee_link.STL
- added link right_shoulder_pitch_link, mass 0.276; collision mesh filename=meshes/right_shoulder_pitch_link.STL; visual mesh filename=meshes/right_shoulder_pitch_link.STL
- added link right_shoulder_roll_link, mass 1.126; collision mesh filename=meshes/right_shoulder_roll_link.STL; visual mesh filename=meshes/right_shoulder_roll_link.STL
- added link right_shoulder_yaw_link, mass 0.896; collision mesh filename=meshes/right_shoulder_yaw_link.STL; visual mesh filename=meshes/right_shoulder_yaw_link.STL
- added link right_wrist_roll_link, mass 0.692; collision mesh filename=meshes/right_wrist_roll_link.STL; visual mesh filename=meshes/right_wrist_roll_link.STL
- link head_link: mass 1.67 -> 1
- link logo_link: mass 0.00512067007990884 -> 0.01
- link torso_link: mass 0.0051207 -> 11
- link waist_yaw_link: mass 10.129 -> 0.2
Joints:
- removed joint L_ankle_pitch
- removed joint L_elbow_pitch
- removed joint L_hip_pitch
- removed joint L_hip_roll
- removed joint L_hip_yaw
- removed joint L_knee_pitch
- removed joint L_shoulder_pitch
- removed joint L_shoulder_roll
- removed joint L_shoulder_yaw
- removed joint R_ankle_pitch
- removed joint R_elbow_pitch
- removed joint R_hip_pitch
- removed joint R_hip_roll
- removed joint R_hip_yaw
- removed joint R_knee_pitch
- removed joint R_shoulder_pitch
- removed joint R_shoulder_roll
- removed joint R_shoulder_yaw
- removed joint head
- removed joint logo
- added joint head_joint: type fixed, parent torso_link, child head_link, origin xyz=-0.01 0 0.3575 rpy=0 0 0, axis 0 0 0
- added joint left_ankle_pitch_joint: type revolute, parent left_knee_link, child left_ankle_pitch_link, origin xyz=0 0 -0.35 rpy=0 0 0, axis 0 1 0, limit lower=-1.047 upper=1.047 effort=64.8 velocity=216.66
- added joint left_elbow_joint: type revolute, parent left_shoulder_yaw_link, child left_elbow_link, origin xyz=0.01 0 -0.151 rpy=0 0 0, axis 0 1 0, limit lower=-0.873 upper=1.571 effort=14 velocity=36
- added joint left_hip_pitch_joint: type revolute, parent left_hip_roll_link, child left_hip_pitch_link, origin xyz=0 0 -0.11 rpy=0 0 0, axis 0 1 0, limit lower=-2.094 upper=0.534 effort=212 velocity=58.7
- added joint left_hip_roll_joint: type revolute, parent left_hip_yaw_link, child left_hip_roll_link, origin xyz=0 0.12 -0.001 rpy=0 0 0, axis 1 0 0, limit lower=-0.349 upper=0.534 effort=100 velocity=31
- added joint left_hip_yaw_joint: type revolute, parent pelvis, child left_hip_yaw_link, origin xyz=0 0 -0.1315 rpy=0 0 0, axis 0 0 1, limit lower=-0.785 upper=0.785 effort=50 velocity=51
- added joint left_knee_joint: type revolute, parent left_hip_pitch_link, child left_knee_link, origin xyz=0 0 -0.35 rpy=0 0 0, axis 0 1 0, limit lower=0 upper=2.269 effort=93 velocity=150
- added joint left_shoulder_pitch_joint: type revolute, parent torso_link, child left_shoulder_pitch_link, origin xyz=-0.01 0.13365 0.31135 rpy=0.17453 0 0, axis 0 1 0, limit lower=-2.749 upper=2.749 effort=18 velocity=36
- added joint left_shoulder_roll_joint: type revolute, parent left_shoulder_pitch_link, child left_shoulder_roll_link, origin xyz=0 0.0588 0 rpy=-0.17453 0 0, axis 1 0 0, limit lower=-0.175 upper=2.653 effort=14 velocity=36
- added joint left_shoulder_yaw_joint: type revolute, parent left_shoulder_roll_link, child left_shoulder_yaw_link, origin xyz=0 0.018928 -0.10734 rpy=0.17453 0 0, axis 0 0 1, limit lower=-2.618 upper=2.618 effort=14 velocity=36
- added joint left_wrist_roll_joint: type revolute, parent left_elbow_link, child left_wrist_roll_link, origin xyz=0.201 0 -0.01 rpy=-0.17453 0 0, axis 1 0 0, limit lower=-2.662 upper=2.662 effort=2.2 velocity=36
- added joint logo_joint: type fixed, parent torso_link, child logo_link, origin xyz=0 0 0 rpy=0 0 0, axis 0 0 0
- added joint right_ankle_pitch_joint: type revolute, parent right_knee_link, child right_ankle_pitch_link, origin xyz=0 0 -0.35 rpy=0 -0.0012589 0, axis 0 1 0, limit lower=-1.047 upper=1.047 effort=64.8 velocity=216.66
- added joint right_elbow_joint: type revolute, parent right_shoulder_yaw_link, child right_elbow_link, origin xyz=0.01 0 -0.151 rpy=0 0 0, axis 0 1 0, limit lower=-0.873 upper=1.571 effort=14 velocity=36
- added joint right_hip_pitch_joint: type revolute, parent right_hip_roll_link, child right_hip_pitch_link, origin xyz=0 0 -0.11 rpy=0 0 0, axis 0 1 0, limit lower=-2.094 upper=0.534 effort=212 velocity=58.7
- added joint right_hip_roll_joint: type revolute, parent right_hip_yaw_link, child right_hip_roll_link, origin xyz=0 -0.12 -0.001 rpy=0 0 0, axis 1 0 0, limit lower=-0.534 upper=0.349 effort=100 velocity=31
- added joint right_hip_yaw_joint: type revolute, parent pelvis, child right_hip_yaw_link, origin xyz=0 0 -0.1315 rpy=0 0 0, axis 0 0 1, limit lower=-0.785 upper=0.785 effort=50 velocity=51
- added joint right_knee_joint: type revolute, parent right_hip_pitch_link, child right_knee_link, origin xyz=0 0 -0.35 rpy=0 0 0, axis 0 1 0, limit lower=0 upper=2.269 effort=93 velocity=150
- added joint right_shoulder_pitch_joint: type revolute, parent torso_link, child right_shoulder_pitch_link, origin xyz=-0.01 -0.13365 0.31135 rpy=-0.17453 0 0, axis 0 1 0, limit lower=-2.749 upper=2.749 effort=18 velocity=36
- added joint right_shoulder_roll_joint: type revolute, parent right_shoulder_pitch_link, child right_shoulder_roll_link, origin xyz=0 -0.0588 0 rpy=0.17453 0 0, axis 1 0 0, limit lower=-2.653 upper=0.175 effort=14 velocity=36
- added joint right_shoulder_yaw_joint: type revolute, parent right_shoulder_roll_link, child right_shoulder_yaw_link, origin xyz=0 -0.018928 -0.10734 rpy=-0.17453 0 0, axis 0 0 1, limit lower=-2.618 upper=2.618 effort=14 velocity=36
- added joint right_wrist_roll_joint: type revolute, parent right_elbow_link, child right_wrist_roll_link, origin xyz=0.201 0 -0.01 rpy=0.17453 0 0, axis 1 0 0, limit lower=-2.662 upper=2.662 effort=2.2 velocity=36
- joint torso: origin xyz=0 0 0.03675 rpy=0 0 0 -> xyz=0 0 0.1315 rpy=0 0 0
- joint waist_yaw: limit lower=-1.047 upper=1.047 effort=60 velocity=43 -> lower=-0.829 upper=0.829 effort=50 velocity=51; origin xyz=0 0 0.08375 rpy=0 0 0 -> xyz=0 0 -0.1315 rpy=0 0 0; parent pelvis_link -> pelvis
